Commit message: added range sensor messages

File: urdf/wild_thumper.urdf.xacro (robot description, xacro)
@@ -5,5 +5,5 @@
 	<link name="base_link">
 		<visual>
-			<origin xyz="0.09 -0.02 0.07" rpy="${PI} 0 ${-PI/2}"/>
+			<origin xyz="0.09 -0.022 0.07" rpy="${PI} 0 ${-PI/2}"/>
 			<geometry>
 				<mesh filename="package://wild_thumper/meshes/wild_thumper_assembly_corrected.stl" scale="0.001 0.001 0.001" />
@@ -34,4 +34,48 @@
 		<origin xyz="0.107 0.0 0.04" rpy="0 0 0"/>
 	</xacro:asus_camera>
+	<link name="sonar_forward">
+		<visual>
+			<geometry>
+				<box size="0.016 0.044 0.02"/>
+			</geometry>
+			<origin xyz="${0.016/2} 0 0" rpy="0 0 0"/>
+			<material name="green">
+				<color rgba="0 1 0 0.8"/>
+			</material>
+		</visual>
+	</link>
+	<link name="sonar_backward">
+		<visual>
+			<geometry>
+				<box size="0.016 0.044 0.02"/>
+			</geometry>
+			<origin xyz="${0.016/2} 0 0" rpy="0 0 0"/>
+			<material name="green">
+				<color rgba="0 1 0 0.8"/>
+			</material>
+		</visual>
+	</link>
+	<link name="ir_left">
+		<visual>
+			<geometry>
+				<box size="0.015 0.015 0.046"/>
+			</geometry>
+			<origin xyz="${-0.015/2} 0 0" rpy="0 0 0"/>
+			<material name="black">
+				<color rgba="0 0 0 1"/>
+			</material>
+		</visual>
+	</link>
+	<link name="ir_right">
+		<visual>
+			<geometry>
+				<box size="0.015 0.015 0.046"/>
+			</geometry>
+			<origin xyz="${-0.015/2} 0 0" rpy="0 0 0"/>
+			<material name="black">
+				<color rgba="0 0 0 1"/>
+			</material>
+		</visual>
+	</link>
 	<joint name="imu_joint" type="fixed">
 		<parent link="base_link"/>
@@ -44,3 +88,23 @@
 		<origin xyz="0.0 0.0 0.13" rpy="0 0 0"/>
 	</joint>
+	<joint name="sonar_forward_joint" type="fixed">
+		<parent link="base_link"/>
+		<child link="sonar_forward"/>
+		<origin xyz="0.115 0.0 -0.012" rpy="0 0 0"/>
+	</joint>
+	<joint name="sonar_backward_joint" type="fixed">
+		<parent link="base_link"/>
+		<child link="sonar_backward"/>
+		<origin xyz="-0.115 0.0 -0.012" rpy="0 ${PI} 0"/>
+	</joint>
+	<joint name="ir_left_joint" type="fixed">
+		<parent link="base_link"/>
+		<child link="ir_left"/>
+		<origin xyz="0.0 ${0.072+0.015} -0.045" rpy="0 0 ${PI/2}"/>
+	</joint>
+	<joint name="ir_right_joint" type="fixed">
+		<parent link="base_link"/>
+		<child link="ir_right"/>
+		<origin xyz="0.0 ${-0.072-0.015} -0.045" rpy="0 0 ${-PI/2}"/>
+	</joint>
 </robot>

Commit message: added robot_pose_ekf

File: urdf/wild_thumper.urdf.xacro (robot description, xacro)
@@ -5,5 +5,5 @@
 	<link name="base_link">
 		<visual>
-			<origin xyz="0.02 0.165 0.2" rpy="${PI} 0 ${-PI/2}"/>
+			<origin xyz="0.09 -0.02 0.07" rpy="${PI} 0 ${-PI/2}"/>
 			<geometry>
 				<mesh filename="package://wild_thumper/meshes/wild_thumper_assembly_corrected.stl" scale="0.001 0.001 0.001" />
@@ -11,6 +11,36 @@
 		</visual>
 	</link>
+	<link name="base_footprint">
+		<visual>
+			<geometry>
+				<box size="0.28 0.31 0.0"/>
+			</geometry>
+			<material name="grey">
+				<color rgba="0.5 0.5 0.5 0.5"/>
+			</material>
+		</visual>
+	</link>
+	<link name="base_imu_link">
+		<visual>
+			<geometry>
+				<box size="0.041 0.028 0.002"/>
+			</geometry>
+			<material name="red">
+				<color rgba="1 0 0 1"/>
+			</material>
+		</visual>
+	</link>
 	<xacro:asus_camera name="camera" parent="base_link">
-		<origin xyz="0 0.19 0.15" rpy="0 0 0"/>
+		<origin xyz="0.107 0.0 0.04" rpy="0 0 0"/>
 	</xacro:asus_camera>
+	<joint name="imu_joint" type="fixed">
+		<parent link="base_link"/>
+		<child link="base_imu_link"/>
+		<origin xyz="0.06 -0.03 0.058" rpy="0 0 0"/>
+	</joint>
+	<joint name="base_link_joint" type="fixed">
+		<parent link="base_footprint"/>
+		<child link="base_link"/>
+		<origin xyz="0.0 0.0 0.13" rpy="0 0 0"/>
+	</joint>
 </robot>

Commit message: urdf: fix elements rotation

File: urdf/wild_thumper.urdf.xacro (robot description, xacro)
@@ -5,5 +5,5 @@
 	<link name="base_link">
 		<visual>
-			<origin xyz="0.02 0.165 0.2" rpy="${PI} 0 0"/>
+			<origin xyz="0.02 0.165 0.2" rpy="${PI} 0 ${-PI/2}"/>
 			<geometry>
 				<mesh filename="package://wild_thumper/meshes/wild_thumper_assembly_corrected.stl" scale="0.001 0.001 0.001" />
@@ -12,5 +12,5 @@
 	</link>
 	<xacro:asus_camera name="camera" parent="base_link">
-		<origin xyz="0 0.19 0.15" rpy="0 0 ${PI/2}"/>
+		<origin xyz="0 0.19 0.15" rpy="0 0 0"/>
 	</xacro:asus_camera>
 </robot>

Commit message: cut 6wd model to 4wd

File: urdf/wild_thumper.urdf.xacro (robot description, xacro)
@@ -5,7 +5,7 @@
 	<link name="base_link">
 		<visual>
-			<origin xyz="0.09 -0.022 0.07" rpy="${PI} 0 ${-PI/2}"/>
+			<origin xyz="0 0 -0.13" rpy="0 0 0"/>
 			<geometry>
-				<mesh filename="package://wild_thumper/meshes/wild_thumper_assembly_corrected.stl" scale="0.001 0.001 0.001" />
+				<mesh filename="package://wild_thumper/meshes/wild_thumper_4wd.stl" scale="1 1 1" />
 			</geometry>
 		</visual>

Commit message: added gazebo simulation

File: urdf/wild_thumper.urdf.xacro (robot description, xacro)
@@ -1,14 +1,6 @@
 <?xml version="1.0"?>
-<robot name="r2" xmlns:xacro="http://ros.org/wiki/xacro">
+<robot name="wild_thumper" xmlns:xacro="http://ros.org/wiki/xacro">
 	<xacro:property name="PI" value="3.1415926535897931" />
 	<xacro:include filename="$(find hector_sensors_description)/urdf/asus_camera.urdf.xacro" />
-	<link name="base_link">
-		<visual>
-			<origin xyz="0 0 -0.13" rpy="0 0 0"/>
-			<geometry>
-				<mesh filename="package://wild_thumper/meshes/wild_thumper_4wd.stl" scale="1 1 1" />
-			</geometry>
-		</visual>
-	</link>
 	<link name="base_footprint">
 		<visual>
@@ -20,4 +12,20 @@
 			</material>
 		</visual>
+	</link>
+	<link name="base_link">
+		<collision>
+			<geometry>
+				<box size="0.23 0.18 0.09"/>
+			</geometry>
+		</collision>
+		<visual>
+			<geometry>
+				<mesh filename="package://wild_thumper/meshes/wild_thumper_4wd.stl" />
+			</geometry>
+		</visual>
+		<inertial>
+			<mass value="1.9"/>
+			<inertia ixx="1.0" ixy="0.0" ixz="0.0" iyy="1.0" iyz="0.0" izz="1.0"/>
+		</inertial>
 	</link>
 	<link name="base_imu_link">
@@ -31,5 +39,12 @@
 		</visual>
 	</link>
-	<xacro:asus_camera name="camera" parent="base_link">
+	<link name="mounting_plate">
+		<visual>
+			<geometry>
+				<box size="0.23 0.12 0.001"/>
+			</geometry>
+		</visual>
+	</link>
+	<xacro:asus_camera name="camera" parent="mounting_plate">
 		<origin xyz="0.107 0.0 0.04" rpy="0 0 0"/>
 	</xacro:asus_camera>
@@ -78,33 +93,103 @@
 		</visual>
 	</link>
+	<joint name="base_link_joint" type="fixed">
+		<parent link="base_footprint"/>
+		<child link="base_link"/>
+		<origin xyz="0.0 0.0 0.082" rpy="0 0 0"/>
+	</joint>
+	<joint name="mounting_plate_joint" type="fixed">
+		<parent link="base_link"/>
+		<child link="mounting_plate"/>
+		<origin xyz="0.0 0.0 0.044" rpy="0 0 0"/>
+	</joint>
 	<joint name="imu_joint" type="fixed">
-		<parent link="base_link"/>
+		<parent link="mounting_plate"/>
 		<child link="base_imu_link"/>
 		<origin xyz="0.06 -0.03 0.058" rpy="0 0 0"/>
 	</joint>
-	<joint name="base_link_joint" type="fixed">
-		<parent link="base_footprint"/>
-		<child link="base_link"/>
-		<origin xyz="0.0 0.0 0.13" rpy="0 0 0"/>
-	</joint>
 	<joint name="sonar_forward_joint" type="fixed">
-		<parent link="base_link"/>
+		<parent link="mounting_plate"/>
 		<child link="sonar_forward"/>
 		<origin xyz="0.115 0.0 -0.012" rpy="0 0 0"/>
 	</joint>
 	<joint name="sonar_backward_joint" type="fixed">
-		<parent link="base_link"/>
+		<parent link="mounting_plate"/>
 		<child link="sonar_backward"/>
 		<origin xyz="-0.115 0.0 -0.012" rpy="0 ${PI} 0"/>
 	</joint>
 	<joint name="ir_left_joint" type="fixed">
-		<parent link="base_link"/>
+		<parent link="mounting_plate"/>
 		<child link="ir_left"/>
 		<origin xyz="0.0 ${0.072+0.015} -0.045" rpy="0 0 ${PI/2}"/>
 	</joint>
 	<joint name="ir_right_joint" type="fixed">
-		<parent link="base_link"/>
+		<parent link="mounting_plate"/>
 		<child link="ir_right"/>
 		<origin xyz="0.0 ${-0.072-0.015} -0.045" rpy="0 0 ${-PI/2}"/>
 	</joint>
+	<xacro:macro name="wheel" params="pos side xyz rpy">
+		<link name="${pos}_${side}_wheel">
+			<visual>
+				<origin xyz="0 0 0" rpy="0 0 0"/>
+				<geometry>
+					<mesh filename="package://wild_thumper/meshes/wheel_${side}.stl" />
+				</geometry>
+			</visual>
+			<collision>
+				<origin xyz="0 0 0" rpy="${-PI/2} 0 0"/>
+				<geometry>
+					<cylinder radius="0.06" length="0.06"/>
+				</geometry>
+			</collision>
+			<inertial>
+				<origin xyz="0 0 0" rpy="0 0 0"/>
+				<mass value="0.1"/>
+				<inertia ixx="0.01" ixy="0" ixz="0" iyy="0.01" iyz="0" izz="0.01"/>
+			</inertial>
+		</link>
+		<joint name="${pos}_${side}_wheel_joint" type="continuous">
+			<parent link="base_link"/>
+			<child link="${pos}_${side}_wheel"/>
+			<axis xyz="0 1 0"/>
+			<origin xyz="${xyz}" rpy="${rpy}"/>
+		</joint>
+	</xacro:macro>
+	<gazebo reference="front_left_wheel">
+		<dampingFactor>0.001</dampingFactor>
+	</gazebo>
+	<gazebo reference="front_right_wheel">
+		<dampingFactor>0.001</dampingFactor>
+	</gazebo>
+	<xacro:wheel pos="aft" side="left"  xyz="-0.06398 0.11407 -0.022446" rpy="0 0 0" />
+	<xacro:wheel pos="aft" side="right" xyz="-0.07397 -0.11408 -0.022446" rpy="0 0 0" />
+	<xacro:wheel pos="front" side="left"  xyz="0.07602 0.11407 -0.022446" rpy="0 0 0" />
+	<xacro:wheel pos="front" side="right" xyz="0.07397 -0.11408 -0.022446" rpy="0 0 0" />
+	<gazebo>
+		<plugin name="joint_state_publisher" filename="libgazebo_ros_joint_state_publisher.so">
+			<robotNamespace>/</robotNamespace>
+			<jointName>aft_left_wheel_joint, aft_right_wheel_joint, front_left_wheel_joint, front_right_wheel_joint</jointName>
+			<updateRate>10.0</updateRate>
+			<alwaysOn>true</alwaysOn>
+		</plugin>
+		<plugin name="differential_drive_controller" filename="libgazebo_ros_diff_drive.so">
+			<robotNamespace>/</robotNamespace>
+			<alwaysOn>true</alwaysOn>
+			<updateRate>10.0</updateRate>
+			<leftJoint>aft_right_wheel_joint</leftJoint>
+			<rightJoint>aft_left_wheel_joint</rightJoint>
+			<wheelSeparation>0.252</wheelSeparation>
+			<wheelDiameter>0.12</wheelDiameter>
+			<wheelTorque>5.0</wheelTorque>
+			<commandTopic>cmd_vel</commandTopic>
+			<odometryTopic>odom</odometryTopic>
+			<odometryFrame>odom</odometryFrame>
+			<robotBaseFrame>base_footprint</robotBaseFrame>
+			<rosDebugLevel>Info</rosDebugLevel>
+			<publishWheelTF>false</publishWheelTF>
+			<publishWheelJointState>true</publishWheelJointState>
+			<wheelAcceleration>0.0</wheelAcceleration>
+			<odometrySource>world</odometrySource>
+			<publishTf>true</publishTf>
+		</plugin>
+	</gazebo>
 </robot>

Commit message: simulation/gazebo: added controller for imu, range sensors and diff drive

File: urdf/wild_thumper.urdf.xacro (robot description, xacro)
@@ -25,5 +25,5 @@
 		</visual>
 		<inertial>
-			<mass value="1.9"/>
+			<mass value="2.5"/>
 			<inertia ixx="1.0" ixy="0.0" ixz="0.0" iyy="1.0" iyz="0.0" izz="1.0"/>
 		</inertial>
@@ -154,42 +154,77 @@
 			<origin xyz="${xyz}" rpy="${rpy}"/>
 		</joint>
+		<transmission name="${pos}_${side}_wheel_trans" type="SimpleTransmission">
+			<type>transmission_interface/SimpleTransmission</type>
+			<joint name="${pos}_${side}_wheel_joint">
+				<hardwareInterface>VelocityJointInterface</hardwareInterface>
+			</joint>
+			<actuator name="{pos}_${side}_wheel_motor">
+				<hardwareInterface>VelocityJointInterface</hardwareInterface>
+				<mechanicalReduction>1</mechanicalReduction>
+			</actuator>
+		</transmission>
 	</xacro:macro>
-	<gazebo reference="front_left_wheel">
-		<dampingFactor>0.001</dampingFactor>
-	</gazebo>
-	<gazebo reference="front_right_wheel">
-		<dampingFactor>0.001</dampingFactor>
-	</gazebo>
-	<xacro:wheel pos="aft" side="left"  xyz="-0.06398 0.11407 -0.022446" rpy="0 0 0" />
-	<xacro:wheel pos="aft" side="right" xyz="-0.07397 -0.11408 -0.022446" rpy="0 0 0" />
-	<xacro:wheel pos="front" side="left"  xyz="0.07602 0.11407 -0.022446" rpy="0 0 0" />
-	<xacro:wheel pos="front" side="right" xyz="0.07397 -0.11408 -0.022446" rpy="0 0 0" />
+	<xacro:wheel pos="rear" side="left"  xyz="-0.06398 0.114 -0.022446" rpy="0 0 0" />
+	<xacro:wheel pos="rear" side="right" xyz="-0.07397 -0.114 -0.022446" rpy="0 0 0" />
+	<xacro:wheel pos="front" side="left"  xyz="0.07602 0.114 -0.022446" rpy="0 0 0" />
+	<xacro:wheel pos="front" side="right" xyz="0.07397 -0.114 -0.022446" rpy="0 0 0" />
 	<gazebo>
-		<plugin name="joint_state_publisher" filename="libgazebo_ros_joint_state_publisher.so">
+		<plugin name="gazebo_ros_control" filename="libgazebo_ros_control.so">
 			<robotNamespace>/</robotNamespace>
-			<jointName>aft_left_wheel_joint, aft_right_wheel_joint, front_left_wheel_joint, front_right_wheel_joint</jointName>
-			<updateRate>10.0</updateRate>
+			<robotSimType>gazebo_ros_control/DefaultRobotHWSim</robotSimType>
+		</plugin>
+		<plugin name="imu_controller" filename="libgazebo_ros_imu.so">
 			<alwaysOn>true</alwaysOn>
-		</plugin>
-		<plugin name="differential_drive_controller" filename="libgazebo_ros_diff_drive.so">
-			<robotNamespace>/</robotNamespace>
-			<alwaysOn>true</alwaysOn>
-			<updateRate>10.0</updateRate>
-			<leftJoint>aft_right_wheel_joint</leftJoint>
-			<rightJoint>aft_left_wheel_joint</rightJoint>
-			<wheelSeparation>0.252</wheelSeparation>
-			<wheelDiameter>0.12</wheelDiameter>
-			<wheelTorque>5.0</wheelTorque>
-			<commandTopic>cmd_vel</commandTopic>
-			<odometryTopic>odom</odometryTopic>
-			<odometryFrame>odom</odometryFrame>
-			<robotBaseFrame>base_footprint</robotBaseFrame>
-			<rosDebugLevel>Info</rosDebugLevel>
-			<publishWheelTF>false</publishWheelTF>
-			<publishWheelJointState>true</publishWheelJointState>
-			<wheelAcceleration>0.0</wheelAcceleration>
-			<odometrySource>world</odometrySource>
-			<publishTf>true</publishTf>
+			<updateRate>20.0</updateRate>
+			<bodyName>base_imu_link</bodyName>
+			<topicName>imu</topicName>
+			<gaussianNoise>0.05</gaussianNoise>
+			<frameName>base_imu_link</frameName>
+			<xyzOffsets>0 0 0</xyzOffsets>
+			<rpyOffset>0 0 0</rpyOffset>
 		</plugin>
 	</gazebo>
+	<xacro:macro name="range_sensor" params="name ros_topic update_rate minRange maxRange fov radiation">
+		<gazebo reference="${name}">
+			<sensor type="ray" name="${name}_sensor">
+				<pose>0 0 0 0 0 0</pose>
+				<update_rate>${update_rate}</update_rate>
+				<visualize>false</visualize>
+				<ray>
+					<scan>
+						<horizontal>
+							<samples>5</samples>
+							<resolution>1</resolution>
+							<min_angle>-${fov/2}</min_angle>
+							<max_angle>${fov/2}</max_angle>
+						</horizontal>
+						<vertical>
+							<samples>5</samples>
+							<resolution>1</resolution>
+							<min_angle>-${fov/2}</min_angle>
+							<max_angle>${fov/2}</max_angle>
+						</vertical>
+					</scan>
+					<range>
+						<min>${minRange}</min>
+						<max>${maxRange}</max>
+						<resolution>0.01</resolution>
+					</range>
+				</ray>
+				<plugin filename="libgazebo_ros_range.so" name="gazebo_ros_range">
+					<gaussianNoise>0.005</gaussianNoise>
+					<alwaysOn>true</alwaysOn>
+					<updateRate>${update_rate}</updateRate>
+					<topicName>${ros_topic}</topicName>
+					<frameName>${name}</frameName>
+					<fov>${fov}</fov>
+					<radiation>${radiation}</radiation>
+				</plugin>
+			</sensor>
+		</gazebo>
+	</xacro:macro>
+	<xacro:range_sensor name="sonar_forward" ros_topic="range_forward" update_rate="10" minRange="0.04" maxRange="6" fov="${60*PI/180}" radiation="ultrasound" />
+	<xacro:range_sensor name="sonar_backward" ros_topic="range_backward" update_rate="10" minRange="0.04" maxRange="6" fov="${60*PI/180}" radiation="ultrasound" />
+	<xacro:range_sensor name="ir_left" ros_topic="range_left" update_rate="10" minRange="0.04" maxRange="0.3" fov="${5*PI/180}" radiation="infrared" />
+	<xacro:range_sensor name="ir_right" ros_topic="range_right" update_rate="10" minRange="0.04" maxRange="0.3" fov="${5*PI/180}" radiation="infrared" />
 </robot>

Commit message: exploration tuning

File: urdf/wild_thumper.urdf.xacro (robot description, xacro)
@@ -6,5 +6,5 @@
 		<visual>
 			<geometry>
-				<box size="0.28 0.31 0.0"/>
+				<box size="0.28 0.31 0.000001"/>
 			</geometry>
 			<material name="grey">

Commit message: fix simulation

File: urdf/wild_thumper.urdf.xacro (robot description, xacro)
@@ -20,4 +20,5 @@
 		</collision>
 		<visual>
+			<origin xyz="-0.00275 0 0" rpy="0 0 0"/>
 			<geometry>
 				<mesh filename="package://wild_thumper/meshes/wild_thumper_4wd.stl" />
@@ -25,4 +26,5 @@
 		</visual>
 		<inertial>
+			<origin xyz="-0.00275 0 -0.02" rpy="0 0 0"/>
 			<mass value="2.5"/>
 			<inertia ixx="1.0" ixy="0.0" ixz="0.0" iyy="1.0" iyz="0.0" izz="1.0"/>
@@ -145,7 +147,14 @@
 				<origin xyz="0 0 0" rpy="0 0 0"/>
 				<mass value="0.1"/>
-				<inertia ixx="0.01" ixy="0" ixz="0" iyy="0.01" iyz="0" izz="0.01"/>
+				<inertia ixx="0.005" ixy="0" ixz="0" iyy="0.005" iyz="0" izz="0.005"/>
 			</inertial>
 		</link>
+		<gazebo reference="${pos}_${side}_wheel">
+			<mu1 value="1.0"/>
+			<mu2 value="1.0"/>
+			<kp value="1000000.0" />
+			<kd value="1.0" />
+			<fdir1 value="1 0 0"/>
+		</gazebo>
 		<joint name="${pos}_${side}_wheel_joint" type="continuous">
 			<parent link="base_link"/>
@@ -160,13 +169,12 @@
 			</joint>
 			<actuator name="{pos}_${side}_wheel_motor">
-				<hardwareInterface>VelocityJointInterface</hardwareInterface>
 				<mechanicalReduction>1</mechanicalReduction>
 			</actuator>
 		</transmission>
 	</xacro:macro>
-	<xacro:wheel pos="rear" side="left"  xyz="-0.06398 0.114 -0.022446" rpy="0 0 0" />
-	<xacro:wheel pos="rear" side="right" xyz="-0.07397 -0.114 -0.022446" rpy="0 0 0" />
-	<xacro:wheel pos="front" side="left"  xyz="0.07602 0.114 -0.022446" rpy="0 0 0" />
-	<xacro:wheel pos="front" side="right" xyz="0.07397 -0.114 -0.022446" rpy="0 0 0" />
+	<xacro:wheel pos="rear" side="left"   xyz="-0.07525  0.12 -0.025" rpy="${-5*PI/180} 0 0" />
+	<xacro:wheel pos="rear" side="right"  xyz="-0.07525 -0.12 -0.025" rpy="${5*PI/180} 0 0" />
+	<xacro:wheel pos="front" side="left"  xyz=" 0.07525  0.12 -0.025" rpy="${-5*PI/180} 0 0" />
+	<xacro:wheel pos="front" side="right" xyz=" 0.07525 -0.12 -0.025" rpy="${5*PI/180} 0 0" />
 	<gazebo>
 		<plugin name="gazebo_ros_control" filename="libgazebo_ros_control.so">
@@ -183,4 +191,5 @@
 			<xyzOffsets>0 0 0</xyzOffsets>
 			<rpyOffset>0 0 0</rpyOffset>
+			<serviceName>/default_imu</serviceName>
 		</plugin>
 	</gazebo>
@@ -224,6 +233,6 @@
 		</gazebo>
 	</xacro:macro>
-	<xacro:range_sensor name="sonar_forward" ros_topic="range_forward" update_rate="10" minRange="0.04" maxRange="6" fov="${30*PI/180}" radiation="ultrasound" />
-	<xacro:range_sensor name="sonar_backward" ros_topic="range_backward" update_rate="10" minRange="0.04" maxRange="6" fov="${30*PI/180}" radiation="ultrasound" />
+	<xacro:range_sensor name="sonar_forward" ros_topic="range_forward" update_rate="10" minRange="0.04" maxRange="0.5" fov="${20*PI/180}" radiation="ultrasound" />
+	<xacro:range_sensor name="sonar_backward" ros_topic="range_backward" update_rate="10" minRange="0.04" maxRange="0.5" fov="${20*PI/180}" radiation="ultrasound" />
 	<xacro:range_sensor name="ir_left" ros_topic="range_left" update_rate="10" minRange="0.04" maxRange="0.3" fov="${5*PI/180}" radiation="infrared" />
 	<xacro:range_sensor name="ir_right" ros_topic="range_right" update_rate="10" minRange="0.04" maxRange="0.3" fov="${5*PI/180}" radiation="infrared" />

Commit message: Add third sonar to ros config

File: urdf/wild_thumper.urdf.xacro (robot description, xacro)
@@ -51,5 +51,16 @@
 		<origin xyz="0.107 0.0 0.04" rpy="0 0 0"/>
 	</xacro:asus_camera>
-	<link name="sonar_forward">
+	<link name="sonar_forward_left">
+		<visual>
+			<geometry>
+				<box size="0.016 0.044 0.02"/>
+			</geometry>
+			<origin xyz="${0.016/2} 0 0" rpy="0 0 0"/>
+			<material name="green">
+				<color rgba="0 1 0 0.8"/>
+			</material>
+		</visual>
+	</link>
+	<link name="sonar_forward_right">
 		<visual>
 			<geometry>
@@ -110,8 +121,13 @@
 		<origin xyz="0.06 -0.03 0.058" rpy="0 0 0"/>
 	</joint>
-	<joint name="sonar_forward_joint" type="fixed">
-		<parent link="mounting_plate"/>
-		<child link="sonar_forward"/>
-		<origin xyz="0.115 0.0 -0.012" rpy="0 0 0"/>
+	<joint name="sonar_forward_left_joint" type="fixed">
+		<parent link="mounting_plate"/>
+		<child link="sonar_forward_left"/>
+		<origin xyz="0.115 -0.04 -0.012" rpy="0 0 0"/>
+	</joint>
+	<joint name="sonar_forward_right_joint" type="fixed">
+		<parent link="mounting_plate"/>
+		<child link="sonar_forward_right"/>
+		<origin xyz="0.115 0.04 -0.012" rpy="0 0 0"/>
 	</joint>
 	<joint name="sonar_backward_joint" type="fixed">

Commit message: fixes third sonar integration

File: urdf/wild_thumper.urdf.xacro (robot description, xacro)
@@ -124,10 +124,10 @@
 		<parent link="mounting_plate"/>
 		<child link="sonar_forward_left"/>
+		<origin xyz="0.115 0.04 -0.012" rpy="0 0 0"/>
+	</joint>
+	<joint name="sonar_forward_right_joint" type="fixed">
+		<parent link="mounting_plate"/>
+		<child link="sonar_forward_right"/>
 		<origin xyz="0.115 -0.04 -0.012" rpy="0 0 0"/>
-	</joint>
-	<joint name="sonar_forward_right_joint" type="fixed">
-		<parent link="mounting_plate"/>
-		<child link="sonar_forward_right"/>
-		<origin xyz="0.115 0.04 -0.012" rpy="0 0 0"/>
 	</joint>
 	<joint name="sonar_backward_joint" type="fixed">

Commit message: Move forward sonars 2cm more apart

File: urdf/wild_thumper.urdf.xacro (robot description, xacro)
@@ -124,10 +124,10 @@
 		<parent link="mounting_plate"/>
 		<child link="sonar_forward_left"/>
-		<origin xyz="0.115 0.04 -0.012" rpy="0 0 0"/>
+		<origin xyz="0.115 0.05 -0.012" rpy="0 0 0"/>
 	</joint>
 	<joint name="sonar_forward_right_joint" type="fixed">
 		<parent link="mounting_plate"/>
 		<child link="sonar_forward_right"/>
-		<origin xyz="0.115 -0.04 -0.012" rpy="0 0 0"/>
+		<origin xyz="0.115 -0.05 -0.012" rpy="0 0 0"/>
 	</joint>
 	<joint name="sonar_backward_joint" type="fixed">

Commit message: Set sonar angle to 5° degree

File: urdf/wild_thumper.urdf.xacro (robot description, xacro)
@@ -124,15 +124,15 @@
 		<parent link="mounting_plate"/>
 		<child link="sonar_forward_left"/>
-		<origin xyz="0.115 0.05 -0.012" rpy="0 0 0"/>
+		<origin xyz="0.115 0.05 -0.012" rpy="0 ${-5*PI/180} 0"/>
 	</joint>
 	<joint name="sonar_forward_right_joint" type="fixed">
 		<parent link="mounting_plate"/>
 		<child link="sonar_forward_right"/>
-		<origin xyz="0.115 -0.05 -0.012" rpy="0 0 0"/>
+		<origin xyz="0.115 -0.05 -0.012" rpy="0 ${-5*PI/180} 0"/>
 	</joint>
 	<joint name="sonar_backward_joint" type="fixed">
 		<parent link="mounting_plate"/>
 		<child link="sonar_backward"/>
-		<origin xyz="-0.115 0.0 -0.012" rpy="0 ${PI} 0"/>
+		<origin xyz="-0.115 0.0 -0.012" rpy="0 ${-175*PI/180} 0"/>
 	</joint>
 	<joint name="ir_left_joint" type="fixed">
